File: kicad/secondary_side.kicad_sch (KiCad schematic)
At the start: 54 parts, among them U1 B179, U3 LM324

Commit message: Update schematic
Connections:
- net GND2: now also R36.2, V15.1 (K)
- net Pin 10: now also R36.1; no longer R36.2
- net VDD: now reaches *.1, *.1 (K), *.2 (A), R17.2, R34.2, R46.1, R47.2
- removed net Pin 16/4/5: R36.1, V15.1 (K)
- net V2 renamed VCC
Other:
- moved on the sheet: *, C12, C13, C15, C9, N2, R17, R20, R201, R22, R23, R24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

Commit message: Update schematic
Parts:
- added U2: B179, Package_DIP:DIP-4_W7.62mm, symbol Isolator:EL817
- R18: value R -> 0.22R MAYBE?
- R25: value R -> 1k
Connections:
- net GND2: now also R26.2, R27.2, U2.2; no longer R26.1, R27.1, U3.5 (+)
- net VDD: now also V16.1 (K)
- net at R43.1: now also U2.1
- net at R43.2: now also V16.2 (A)
- net at *.2 (A), C9.1: now also TR1_*L4.5; no longer TR1_*L4.6
- net L4_6 renamed GND1
- net GND1: now also R26.1, R27.1, TR1_*L4.6; no longer R26.2, R27.2, TR1_*L4.5
- new net BAT-: U3.5 (+)
Other:
- moved on the sheet: *, C12, C13, C14, C15, C8, C9, N2, R12, R16, R17, R18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
